File: Pico Speaker EAGLE/picospeaker.sch (EAGLE design)
At the start: 9 parts, among them J1 SPK -/+ MAX 3W, J2 POWER -/+ 4,5v

Commit message: Updates
Parts:
- U$1: value RASPBERRY-PI-PICO_TH -> RASPBERRY-PI-PICO; device pipico:RASPBERRY-PI-PICO_TH -> Proper-Pico:RASPBERRY-PI-PICO
Connections:
- net N$10: now also U$1.GP19; no longer U$1.25
- net N$11: now also U$1.VSYS; no longer U$1.39
- net N$13: now also U$1.GND8; no longer U$1.38
- net N$2: now also U$1.GP21; no longer U$1.27
- net N$3: now also U$1.3V3(OUT); no longer U$1.36
- net N$6: now also U$1.GP0; no longer U$1.1
- net N$7: now also U$1.GP1; no longer U$1.2
- net N$8: now also U$1.GND5; no longer U$1.23
- net N$9: now also U$1.GP20; no longer U$1.26
Other:
- moved on the sheet: R1
Changed lines of the file:
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@@
 </classes>
 <parts>
-<part name="U$1" library="pipico" deviceset="RASPBERRY-PI-PICO_TH" device=""/>
 <part name="U$2" library="DFPlayer_v1" deviceset="DFPLAYER" device=""/>
 <part name="R1" library="SparkFun-Resistors" library_urn="urn:adsk.eagle:library:532" deviceset="1KOHM" device="-HORIZ_KIT-1/4W-5%" package3d_urn="urn:adsk.eagle:package:39661/2" value="1k"/>
@@
 <part name="J2" library="SparkFun-Connectors" library_urn="urn:adsk.eagle:library:513" deviceset="CONN_02" device="" package3d_urn="urn:adsk.eagle:package:38039/2" value="POWER -/+ 4,5v"/>
 <part name="S4" library="SparkFun-Retired" deviceset="SWITCH-SPDT" device="SMD"/>
+<part name="U$1" library="Proper-Pico" deviceset="RASPBERRY-PI-PICO" device=""/>
 </parts>
 <sheets>
@@
 </plain>
 <instances>
-<instance part="U$1" gate="G$1" x="-22.86" y="48.26" smashed="yes"/>
-<instance part="U$2" gate="G$1" x="-22.86" y="93.98" smashed="yes"/>
-<instance part="R1" gate="G$1" x="-48.26" y="101.6" smashed="yes" rot="R180">
-<attribute name="NAME" x="-48.26" y="100.076" size="1.778" layer="95" font="vector" rot="R180" align="bottom-center"/>
-<attribute name="VALUE" x="-48.26" y="103.124" size="1.778" layer="96" font="vector" rot="R180" align="top-center"/>
+<instance part="U$2" gate="G$1" x="-25.4" y="93.98" smashed="yes"/>
+<instance part="R1" gate="G$1" x="-50.8" y="101.6" smashed="yes" rot="R180">
+<attribute name="NAME" x="-50.8" y="100.076" size="1.778" layer="95" font="vector" rot="R180" align="bottom-center"/>
+<attribute name="VALUE" x="-50.8" y="103.124" size="1.778" layer="96" font="vector" rot="R180" align="top-center"/>
 </instance>
 <instance part="J1" gate="J1" x="-55.88" y="86.36" smashed="yes">
@@
 <attribute name="VALUE" x="-2.54" y="77.47" size="1.778" layer="96"/>
 </instance>
+<instance part="U$1" gate="G$1" x="-25.4" y="48.26" smashed="yes"/>
 </instances>
 <busses>
@@
 <pinref part="U$2" gate="G$1" pin="RX"/>
 <pinref part="R1" gate="G$1" pin="1"/>
-<wire x1="-43.18" y1="101.6" x2="-40.64" y2="101.6" width="0.1524" layer="91"/>
+<wire x1="-45.72" y1="101.6" x2="-43.18" y2="101.6" width="0.1524" layer="91"/>
 </segment>
 </net>
 <net name="N$3" class="0">
 <segment>
-<pinref part="U$1" gate="G$1" pin="36"/>
 <wire x1="-7.62" y1="63.5" x2="27.94" y2="63.5" width="0.1524" layer="91"/>
 <wire x1="27.94" y1="63.5" x2="27.94" y2="111.76" width="0.1524" layer="91"/>
-<wire x1="27.94" y1="111.76" x2="-40.64" y2="111.76" width="0.1524" layer="91"/>
+<wire x1="27.94" y1="111.76" x2="-43.18" y2="111.76" width="0.1524" layer="91"/>
 <pinref part="U$2" gate="G$1" pin="VCC"/>
-<wire x1="-40.64" y1="111.76" x2="-40.64" y2="104.14" width="0.1524" layer="91"/>
+<wire x1="-43.18" y1="111.76" x2="-43.18" y2="104.14" width="0.1524" layer="91"/>
+<pinref part="U$1" gate="G$1" pin="3V3(OUT)"/>
 </segment>
 </net>
@@
 <wire x1="-48.26" y1="88.9" x2="-48.26" y2="91.44" width="0.1524" layer="91"/>
 <pinref part="U$2" gate="G$1" pin="SPK_1"/>
-<wire x1="-48.26" y1="91.44" x2="-40.64" y2="91.44" width="0.1524" layer="91"/>
+<wire x1="-48.26" y1="91.44" x2="-43.18" y2="91.44" width="0.1524" layer="91"/>
 </segment>
 </net>
@@
 <pinref part="J1" gate="J1" pin="1"/>
 <pinref part="U$2" gate="G$1" pin="SPK_2"/>
-<wire x1="-48.26" y1="86.36" x2="-40.64" y2="86.36" width="0.1524" layer="91"/>
+<wire x1="-48.26" y1="86.36" x2="-43.18" y2="86.36" width="0.1524" layer="91"/>
 </segment>
 </net>
@@
 <segment>
 <pinref part="R1" gate="G$1" pin="2"/>
-<wire x1="-53.34" y1="101.6" x2="-68.58" y2="101.6" width="0.1524" layer="91"/>
-<pinref part="U$1" gate="G$1" pin="1"/>
+<wire x1="-55.88" y1="101.6" x2="-68.58" y2="101.6" width="0.1524" layer="91"/>
 <wire x1="-68.58" y1="101.6" x2="-68.58" y2="73.66" width="0.1524" layer="91"/>
-<wire x1="-68.58" y1="73.66" x2="-38.1" y2="73.66" width="0.1524" layer="91"/>
+<wire x1="-68.58" y1="73.66" x2="-43.18" y2="73.66" width="0.1524" layer="91"/>
+<pinref part="U$1" gate="G$1" pin="GP0"/>
 </segment>
 </net>
@@
 <segment>
 <pinref part="U$2" gate="G$1" pin="TX"/>
-<wire x1="-40.64" y1="99.06" x2="-66.04" y2="99.06" width="0.1524" layer="91"/>
-<pinref part="U$1" gate="G$1" pin="2"/>
+<wire x1="-43.18" y1="99.06" x2="-66.04" y2="99.06" width="0.1524" layer="91"/>
 <wire x1="-66.04" y1="99.06" x2="-66.04" y2="71.12" width="0.1524" layer="91"/>
-<wire x1="-66.04" y1="71.12" x2="-38.1" y2="71.12" width="0.1524" layer="91"/>
+<wire x1="-66.04" y1="71.12" x2="-43.18" y2="71.12" width="0.1524" layer="91"/>
+<pinref part="U$1" gate="G$1" pin="GP1"/>
 </segment>
 </net>
@@
 <wire x1="-5.08" y1="25.4" x2="33.02" y2="25.4" width="0.1524" layer="91"/>
 <wire x1="33.02" y1="25.4" x2="33.02" y2="88.9" width="0.1524" layer="91"/>
-<wire x1="-5.08" y1="88.9" x2="33.02" y2="88.9" width="0.1524" layer="91"/>
+<wire x1="-7.62" y1="88.9" x2="33.02" y2="88.9" width="0.1524" layer="91"/>
 <pinref part="S1" gate="G$1" pin="1"/>
 <pinref part="S2" gate="G$1" pin="1"/>
@@
 <wire x1="7.62" y1="38.1" x2="7.62" y2="43.18" width="0.1524" layer="91"/>
 <junction x="7.62" y="38.1"/>
-<pinref part="U$1" gate="G$1" pin="23"/>
 <wire x1="-5.08" y1="30.48" x2="-7.62" y2="30.48" width="0.1524" layer="91"/>
 <junction x="-5.08" y="30.48"/>
+<pinref part="U$1" gate="G$1" pin="GND5"/>
 </segment>
 </net>
 <net name="N$2" class="0">
 <segment>
-<pinref part="U$1" gate="G$1" pin="27"/>
 <wire x1="-7.62" y1="40.64" x2="-2.54" y2="40.64" width="0.1524" layer="91"/>
 <pinref part="S3" gate="G$1" pin="2"/>
 <wire x1="-2.54" y1="40.64" x2="-2.54" y2="43.18" width="0.1524" layer="91"/>
+<pinref part="U$1" gate="G$1" pin="GP21"/>
 </segment>
 </net>
 <net name="N$9" class="0">
 <segment>
-<pinref part="U$1" gate="G$1" pin="26"/>
 <pinref part="S2" gate="G$1" pin="2"/>
 <wire x1="-7.62" y1="38.1" x2="-2.54" y2="38.1" width="0.1524" layer="91"/>
+<pinref part="U$1" gate="G$1" pin="GP20"/>
 </segment>
 </net>
 <net name="N$10" class="0">
 <segment>
-<pinref part="U$1" gate="G$1" pin="25"/>
 <wire x1="-7.62" y1="35.56" x2="-2.54" y2="35.56" width="0.1524" layer="91"/>
 <pinref part="S1" gate="G$1" pin="2"/>
 <wire x1="-2.54" y1="35.56" x2="-2.54" y2="33.02" width="0.1524" layer="91"/>
+<pinref part="U$1" gate="G$1" pin="GP19"/>
 </segment>
 </net>
 <net name="N$11" class="0">
 <segment>
-<pinref part="U$1" gate="G$1" pin="39"/>
 <pinref part="S4" gate="1" pin="P"/>
 <wire x1="-7.62" y1="71.12" x2="-2.54" y2="71.12" width="0.1524" layer="91"/>
 <wire x1="-2.54" y1="71.12" x2="-2.54" y2="73.66" width="0.1524" layer="91"/>
+<pinref part="U$1" gate="G$1" pin="VSYS"/>
 </segment>
 </net>
 <net name="N$13" class="0">
 <segment>
-<pinref part="U$1" gate="G$1" pin="38"/>
 <pinref part="J2" gate="J1" pin="1"/>
 <wire x1="-7.62" y1="68.58" x2="7.62" y2="68.58" width="0.1524" layer="91"/>
+<pinref part="U$1" gate="G$1" pin="GND8"/>
 </segment>
 </net>
@@
 </sheet>
 </sheets>
+<errors>
+</errors>
 </schematic>
 </drawing>
